File: kicad/toolhead_pcb.kicad_pcb (KiCad board)
At the start: 2 copper layers, 43 x 34.7 mm, 12 parts, among them J1 MAGPROBE, J2 X_ENDSTOP, J3 COOLING_FAN_1, J4 HOTEND_FAN, J5 Conn_02x08_Top_Bottom, J6 COOLING_FAN_2, J7 HOTEND_THERMISTOR, J8 HOTEND_HEATER, J9 EXTRUDER_STEPPER

Commit message: Push alternative design for board
Parts:
- J1, J2, J3, J4, J7: footprint Connector_Molex:Molex_Micro-Fit_3.0_43650-0215_1x02_P3.00mm_Vertical -> Connector_JST:JST_XH_B2B-XH-A_1x02_P2.50mm_Vertical
- J5: footprint Connector_Molex:Molex_Micro-Fit_3.0_43045-1612_2x08_P3.00mm_Vertical -> Connector_Molex:Molex_Micro-Fit_3.0_43045-1600_2x08_P3.00mm_Horizontal
- J6: value COOLING_FAN_2 -> COOLING_FAN_1; footprint Connector_Molex:Molex_Micro-Fit_3.0_43650-0215_1x02_P3.00mm_Vertical -> Connector_JST:JST_XH_B2B-XH-A_1x02_P2.50mm_Vertical
- J8: footprint Connector_Molex:Molex_Micro-Fit_3.0_43650-0215_1x02_P3.00mm_Vertical -> Connector_Molex:Molex_Micro-Fit_3.0_43650-0200_1x02_P3.00mm_Horizontal
- J9: footprint Connector_Molex:Molex_Micro-Fit_3.0_43650-0415_1x04_P3.00mm_Vertical -> Connector_JST:JST_XH_B4B-XH-A_1x04_P2.50mm_Vertical
- moved J8 116.5 mm to (218.5, 79.5), turned to 0 degrees
- moved J7 107.2 mm to (213.0, 86.8), turned to 0 degrees
- moved J9 91.8 mm to (215.0, 95.0), turned to 0 degrees
- moved H2 88.2 mm to (188.5, 87.2), turned to 0 degrees
- moved H1 88.1 mm to (222.0, 87.0), turned to 0 degrees
- moved J3 82.9 mm to (197.0, 95.0), turned to 0 degrees
- moved J6 72.6 mm to (206.0, 95.0), turned to 0 degrees
- moved J4 69.9 mm to (204.0, 86.8), turned to 0 degrees
- moved J5 66.2 mm to (189.2, 79.5), turned to 0 degrees
- moved J2 55.6 mm to (195.0, 86.8), turned to 0 degrees
- moved J1 50.1 mm to (188.0, 95.0), turned to 0 degrees
- moved G*** 39.7 mm to (94.2, 131.5)
Connections:
- J5 pad 1: MAGPROBE- -> MAGPROBE+
- J5 pad 10: X_ENDSTOP+ -> X_ENDSTOP-
- J5 pad 11: COOLING_FAN+ -> COOLING_FAN-
- J5 pad 12: HOTEND_FAN+ -> HOTEND_FAN-
- J5 pad 15: HOTEND_THERMISTOR+ -> HOTEND_THERMISTOR-
- J5 pad 16: HOTEND_HEATER+ -> HOTEND_HEATER-
- J5 pad 2: X_ENDSTOP- -> X_ENDSTOP+
- J5 pad 3: COOLING_FAN- -> COOLING_FAN+
- J5 pad 4: HOTEND_FAN- -> HOTEND_FAN+
- J5 pad 7: HOTEND_THERMISTOR- -> HOTEND_THERMISTOR+
- J5 pad 8: HOTEND_HEATER- -> HOTEND_HEATER+
- J5 pad 9: MAGPROBE+ -> MAGPROBE-
- J7 pad 1: HOTEND_THERMISTOR+ -> HOTEND_THERMISTOR-
- J7 pad 2: HOTEND_THERMISTOR- -> HOTEND_THERMISTOR+
- J8 pad 1: HOTEND_HEATER+ -> HOTEND_HEATER-
- J8 pad 2: HOTEND_HEATER- -> HOTEND_HEATER+
Routing:
- net HOTEND_FAN-: track 24.9 -> 8.39 mm
- net X_ENDSTOP-: track 19.8 -> 5.39 mm
- net HOTEND_HEATER-: track 8.08 -> 22.2 mm
- net HOTEND_THERMISTOR-: track 19.5 -> 8.24 mm
- net STEPPER_B2: track 23.6 -> 33.2 mm
- net MAGPROBE+: track 8.91 -> 17.9 mm
- net COOLING_FAN-: track 34.5 -> 26.1 mm
- net MAGPROBE-: track 8.08 -> 15.9 mm
- net HOTEND_FAN+: track 20.6 -> 13.3 mm
- net X_ENDSTOP+: track 17.8 -> 10.7 mm
- net STEPPER_B1: track 19.4 -> 26.2 mm
- net COOLING_FAN+: track 40.9 -> 36.2 mm
- net HOTEND_THERMISTOR+: track 17.9 -> 13.3 mm
- net HOTEND_HEATER+: track 8.50 -> 12.9 mm
- net STEPPER_A1: track 22.6 -> 26.6 mm
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- removed copper zone on B.Cu, net (none)
- removed copper zone on F.Cu, net (none)
Other:
- board size 43 x 34.7 mm -> 125.5 x 83.2 mm
- rule pad_to_mask_clearance: 0 -> 0.0508
- rule trace_min: 0.2 -> 0.1524
- rule via_min_drill: 0.2 -> 0.0254
- rule via_min_size: 0.4 -> 0.508
- board text added: "Mantis"
- board text added: "PCB v0.2"
- board text removed: "+"
- board text removed: "-"
- board text removed: "09/2021"
- board text removed: "A"
- board text removed: "A/"
- board text removed: "B"
- board text removed: "B/"
- board text removed: "CF"
- board text removed: "CF1"
- board text removed: "CF2"
- board text removed: "EX"
- board text removed: "HE"
- board text removed: "HF"
- board text removed: "MCU"
- board text removed: "MP"
- board text removed: "PCB v0.1"
- board text removed: "TH"
- board text removed: "XE"
