File: kicad/toolhead_pcb.sch (KiCad schematic (older format))
At the start: 11 parts, among them J1 MAGPROBE, J2 X_ENDSTOP, J3 COOLING_FAN_1, J4 HOTEND_FAN, J5 Conn_02x08_Top_Bottom, J6 COOLING_FAN_2, J7 HOTEND_THERMISTOR, J8 HOTEND_HEATER, J9 EXTRUDER_STEPPER

Commit message: Push alternative design for board
Parts:
- J1, J2, J3, J4, J7: footprint Connector_Molex:Molex_Micro-Fit_3.0_43650-0215_1x02_P3.00mm_Vertical -> Connector_JST:JST_XH_B2B-XH-A_1x02_P2.50mm_Vertical
- J5: footprint Connector_Molex:Molex_Micro-Fit_3.0_43045-1612_2x08_P3.00mm_Vertical -> Connector_Molex:Molex_Micro-Fit_3.0_43045-1600_2x08_P3.00mm_Horizontal
- J6: value COOLING_FAN_2 -> COOLING_FAN_1; footprint Connector_Molex:Molex_Micro-Fit_3.0_43650-0215_1x02_P3.00mm_Vertical -> Connector_JST:JST_XH_B2B-XH-A_1x02_P2.50mm_Vertical
- J8: footprint Connector_Molex:Molex_Micro-Fit_3.0_43650-0215_1x02_P3.00mm_Vertical -> Connector_Molex:Molex_Micro-Fit_3.0_43650-0200_1x02_P3.00mm_Horizontal
- J9: footprint Connector_Molex:Molex_Micro-Fit_3.0_43650-0415_1x04_P3.00mm_Vertical -> Connector_JST:JST_XH_B4B-XH-A_1x04_P2.50mm_Vertical
Connections:
- net COOLING_FAN+: now also J5.3 (Pin_3); no longer J5.11 (Pin_11)
- net COOLING_FAN-: now also J5.11 (Pin_11); no longer J5.3 (Pin_3)
- net HOTEND_FAN+: now also J5.4 (Pin_4); no longer J5.12 (Pin_12)
- net HOTEND_FAN-: now also J5.12 (Pin_12); no longer J5.4 (Pin_4)
- net HOTEND_HEATER+: now also J5.8 (Pin_8), J8.2 (Pin_2); no longer J5.16 (Pin_16), J8.1 (Pin_1)
- net HOTEND_HEATER-: now also J5.16 (Pin_16), J8.1 (Pin_1); no longer J5.8 (Pin_8), J8.2 (Pin_2)
- net HOTEND_THERMISTOR+: now also J5.7 (Pin_7), J7.2 (Pin_2); no longer J5.15 (Pin_15), J7.1 (Pin_1)
- net HOTEND_THERMISTOR-: now also J5.15 (Pin_15), J7.1 (Pin_1); no longer J5.7 (Pin_7), J7.2 (Pin_2)
- net MAGPROBE+: now also J5.1 (Pin_1); no longer J5.9 (Pin_9)
- net MAGPROBE-: now also J5.9 (Pin_9); no longer J5.1 (Pin_1)
- net X_ENDSTOP+: now also J5.2 (Pin_2); no longer J5.10 (Pin_10)
- net X_ENDSTOP-: now also J5.10 (Pin_10); no longer J5.2 (Pin_2)
Changed lines of the file:
@@
 Comment4 ""
 $EndDescr
+Text GLabel 5200 3400 0    50   Input ~ 0
+X_ENDSTOP+
 Text GLabel 5700 3400 2    50   Input ~ 0
-X_ENDSTOP+
-Text GLabel 5200 3400 0    50   Input ~ 0
 X_ENDSTOP-
-Text GLabel 6200 4600 0    50   Input ~ 0
+Text GLabel 6200 4700 0    50   Input ~ 0
 HOTEND_THERMISTOR+
 $Comp
@@
 F 0 "J2" H 4880 4592 50  0000 L CNN
 F 1 "X_ENDSTOP" H 4880 4501 50  0000 L CNN
-F 2 "Connector_Molex:Molex_Micro-Fit_3.0_43650-0215_1x02_P3.00mm_Vertical" H 4800 4600 50  0001 C CNN
+F 2 "Connector_JST:JST_XH_B2B-XH-A_1x02_P2.50mm_Vertical" H 4800 4600 50  0001 C CNN
 F 3 "~" H 4800 4600 50  0001 C CNN
 	1    4800 4600
@@
 F 0 "J3" H 4880 4892 50  0000 L CNN
 F 1 "COOLING_FAN_1" H 4880 4801 50  0000 L CNN
-F 2 "Connector_Molex:Molex_Micro-Fit_3.0_43650-0215_1x02_P3.00mm_Vertical" H 4800 4900 50  0001 C CNN
+F 2 "Connector_JST:JST_XH_B2B-XH-A_1x02_P2.50mm_Vertical" H 4800 4900 50  0001 C CNN
 F 3 "~" H 4800 4900 50  0001 C CNN
 	1    4800 4900
@@
 F 0 "J4" H 4880 5192 50  0000 L CNN
 F 1 "HOTEND_FAN" H 4880 5101 50  0000 L CNN
-F 2 "Connector_Molex:Molex_Micro-Fit_3.0_43650-0215_1x02_P3.00mm_Vertical" H 4800 5200 50  0001 C CNN
+F 2 "Connector_JST:JST_XH_B2B-XH-A_1x02_P2.50mm_Vertical" H 4800 5200 50  0001 C CNN
 F 3 "~" H 4800 5200 50  0001 C CNN
 	1    4800 5200
@@
 P 6400 4300
 F 0 "J6" H 6480 4292 50  0000 L CNN
-F 1 "COOLING_FAN_2" H 6480 4201 50  0000 L CNN
-F 2 "Connector_Molex:Molex_Micro-Fit_3.0_43650-0215_1x02_P3.00mm_Vertical" H 6400 4300 50  0001 C CNN
+F 1 "COOLING_FAN_1" H 6480 4201 50  0000 L CNN
+F 2 "Connector_JST:JST_XH_B2B-XH-A_1x02_P2.50mm_Vertical" H 6400 4300 50  0001 C CNN
 F 3 "~" H 6400 4300 50  0001 C CNN
 	1    6400 4300
@@
 F 0 "J7" H 6480 4592 50  0000 L CNN
 F 1 "HOTEND_THERMISTOR" H 6480 4501 50  0000 L CNN
-F 2 "Connector_Molex:Molex_Micro-Fit_3.0_43650-0215_1x02_P3.00mm_Vertical" H 6400 4600 50  0001 C CNN
+F 2 "Connector_JST:JST_XH_B2B-XH-A_1x02_P2.50mm_Vertical" H 6400 4600 50  0001 C CNN
 F 3 "~" H 6400 4600 50  0001 C CNN
 	1    6400 4600
 	1    0    0    -1
 $EndComp
+Text GLabel 6200 5000 0    50   Input ~ 0
+HOTEND_HEATER+
 Text GLabel 6200 4900 0    50   Input ~ 0
-HOTEND_HEATER+
-Text GLabel 6200 5000 0    50   Input ~ 0
 HOTEND_HEATER-
 Text GLabel 4600 4700 0    50   Input ~ 0
@@
 Text GLabel 4600 4600 0    50   Input ~ 0
 X_ENDSTOP-
-Text GLabel 6200 4700 0    50   Input ~ 0
+Text GLabel 6200 4600 0    50   Input ~ 0
 HOTEND_THERMISTOR-
 Text GLabel 4600 5300 0    50   Input ~ 0
@@
 F 0 "J9" H 6480 5292 50  0000 L CNN
 F 1 "EXTRUDER_STEPPER" H 6480 5201 50  0000 L CNN
-F 2 "Connector_Molex:Molex_Micro-Fit_3.0_43650-0415_1x04_P3.00mm_Vertical" H 6400 5300 50  0001 C CNN
+F 2 "Connector_JST:JST_XH_B4B-XH-A_1x04_P2.50mm_Vertical" H 6400 5300 50  0001 C CNN
 F 3 "~" H 6400 5300 50  0001 C CNN
 	1    6400 5300
@@
 F 0 "J1" H 4880 4292 50  0000 L CNN
 F 1 "MAGPROBE" H 4880 4201 50  0000 L CNN
-F 2 "Connector_Molex:Molex_Micro-Fit_3.0_43650-0215_1x02_P3.00mm_Vertical" H 4800 4300 50  0001 C CNN
+F 2 "Connector_JST:JST_XH_B2B-XH-A_1x02_P2.50mm_Vertical" H 4800 4300 50  0001 C CNN
 F 3 "~" H 4800 4300 50  0001 C CNN
 	1    4800 4300
@@
 F 0 "J8" H 6480 4892 50  0000 L CNN
 F 1 "HOTEND_HEATER" H 6480 4801 50  0000 L CNN
-F 2 "Connector_Molex:Molex_Micro-Fit_3.0_43650-0215_1x02_P3.00mm_Vertical" H 6400 4900 50  0001 C CNN
+F 2 "Connector_Molex:Molex_Micro-Fit_3.0_43650-0200_1x02_P3.00mm_Horizontal" H 6400 4900 50  0001 C CNN
 F 3 "~" H 6400 4900 50  0001 C CNN
 	1    6400 4900
 	1    0    0    -1
 $EndComp
+Text GLabel 5700 3900 2    50   Input ~ 0
+HOTEND_THERMISTOR-
 Text GLabel 5200 3900 0    50   Input ~ 0
-HOTEND_THERMISTOR-
-Text GLabel 5700 3900 2    50   Input ~ 0
 HOTEND_THERMISTOR+
-Text GLabel 5200 4000 0    50   Input ~ 0
+Text GLabel 5700 4000 2    50   Input ~ 0
 HOTEND_HEATER-
-Text GLabel 5200 3300 0    50   Input ~ 0
+Text GLabel 5700 3300 2    50   Input ~ 0
 MAGPROBE-
 Text GLabel 5700 3700 2    50   Input ~ 0
@@
 Text GLabel 5200 3800 0    50   Input ~ 0
 STEPPER_B2
+Text GLabel 5700 3600 2    50   Input ~ 0
+HOTEND_FAN-
+Text GLabel 5700 3500 2    50   Input ~ 0
+COOLING_FAN-
 Text GLabel 5200 3600 0    50   Input ~ 0
-HOTEND_FAN-
+HOTEND_FAN+
 Text GLabel 5200 3500 0    50   Input ~ 0
-COOLING_FAN-
-Text GLabel 5700 3600 2    50   Input ~ 0
-HOTEND_FAN+
-Text GLabel 5700 3500 2    50   Input ~ 0
 COOLING_FAN+
 Text GLabel 5200 3700 0    50   Input ~ 0
@@
 Text GLabel 5700 3800 2    50   Input ~ 0
 STEPPER_B1
-Text GLabel 5700 4000 2    50   Input ~ 0
+Text GLabel 5200 4000 0    50   Input ~ 0
 HOTEND_HEATER+
-Text GLabel 5700 3300 2    50   Input ~ 0
+Text GLabel 5200 3300 0    50   Input ~ 0
 MAGPROBE+
 $Comp
@@
 F 0 "J5" H 5450 4117 50  0000 C CNN
 F 1 "Conn_02x08_Top_Bottom" H 5450 4026 50  0000 C CNN
-F 2 "Connector_Molex:Molex_Micro-Fit_3.0_43045-1612_2x08_P3.00mm_Vertical" H 5400 3600 50  0001 C CNN
+F 2 "Connector_Molex:Molex_Micro-Fit_3.0_43045-1600_2x08_P3.00mm_Horizontal" H 5400 3600 50  0001 C CNN
 F 3 "~" H 5400 3600 50  0001 C CNN
 	1    5400 3600
@@
 $EndComp
 $Comp
-L Mechanical:MountingHole H1
-U 1 1 61360144
-P 4600 5900
-F 0 "H1" H 4700 5946 50  0000 L CNN
-F 1 "MountingHole" H 4700 5855 50  0000 L CNN
-F 2 "MountingHole:MountingHole_3.2mm_M3_ISO7380" H 4600 5900 50  0001 C CNN
-F 3 "~" H 4600 5900 50  0001 C CNN
-	1    4600 5900
+L Mechanical:MountingHole H2
+U 1 1 61375022
+P 5550 5850
+F 0 "H2" H 5650 5896 50  0000 L CNN
+F 1 "MountingHole" H 5650 5805 50  0000 L CNN
+F 2 "MountingHole:MountingHole_3.2mm_M3_ISO7380" H 5550 5850 50  0001 C CNN
+F 3 "~" H 5550 5850 50  0001 C CNN
+	1    5550 5850
 	1    0    0    -1
 $EndComp
 $Comp
-L Mechanical:MountingHole H2
-U 1 1 6136060E
-P 5300 5900
-F 0 "H2" H 5400 5946 50  0000 L CNN
-F 1 "MountingHole" H 5400 5855 50  0000 L CNN
-F 2 "MountingHole:MountingHole_3.2mm_M3_ISO7380" H 5300 5900 50  0001 C CNN
-F 3 "~" H 5300 5900 50  0001 C CNN
-	1    5300 5900
+L Mechanical:MountingHole H1
+U 1 1 61375D63
+P 4650 5850
+F 0 "H1" H 4750 5896 50  0000 L CNN
+F 1 "MountingHole" H 4750 5805 50  0000 L CNN
+F 2 "MountingHole:MountingHole_3.2mm_M3_ISO7380" H 4650 5850 50  0001 C CNN
+F 3 "~" H 4650 5850 50  0001 C CNN
+	1    4650 5850
 	1    0    0    -1
 $EndComp
